File: ESP32USBI2S/ESP32USBI2S.kicad_sch (KiCad schematic)
At the start: 33 parts, among them IC1 TPS7A, IC2 74LVC, IC3 5PB1102, J1 I2S OUT, J2 5V POWER, U1 ESP32-S3, Y2 22.5792MHz, Y3 24.5760Mhz

Commit message: design for bare module
Parts:
- added R1: 0R*, Resistor_SMD:R_0805_2012Metric_Pad1.20x1.40mm_HandSolder, symbol Device:R
- added R11: 10K, Resistor_SMD:R_0603_1608Metric_Pad0.98x0.95mm_HandSolder, symbol Device:R
- C2, C3, C6: value 1uF -> 1uF*
- C5, C7: value 100nF -> 100nF*
- C8, C9: value 220uF -> 220uF*
- IC1: value TPS7A -> TPS7A2033*
- R5: value 0R68 -> 0R68*
Connections:
- net 3V3: now also R1.2, R11.1; no longer IC3.2 (1G)
- net 3V3ESP: now reaches U1.24 (3V3)
- net 3V3ESP: now also R1.1
- new net: IC3.2 (1G), R11.2
Changed lines of the file:
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@@
 	)
 	(junction
+		(at 69.85 45.72)
+		(diameter 0)
+		(color 0 0 0 0)
+	)
+	(junction
 		(at 265.43 64.77)
 		(diameter 0)
@@
 	(wire
 		(pts
-			(xy 67.31 45.72) (xy 72.39 45.72)
+			(xy 67.31 45.72) (xy 69.85 45.72)
 		)
 		(stroke
@@
 	(wire
 		(pts
+			(xy 69.85 45.72) (xy 77.47 45.72)
+		)
+		(stroke
+			(width 0)
+			(type default)
+		)
+	)
+	(wire
+		(pts
 			(xy 209.55 116.84) (xy 220.98 116.84)
 		)
@@
 	(wire
 		(pts
+			(xy 69.85 31.75) (xy 69.85 27.94)
+		)
+		(stroke
+			(width 0)
+			(type default)
+		)
+	)
+	(wire
+		(pts
 			(xy 87.63 59.69) (xy 86.36 59.69)
 		)
@@
 	(wire
 		(pts
+			(xy 142.24 127) (xy 168.91 127)
+		)
+		(stroke
+			(width 0)
+			(type default)
+		)
+	)
+	(wire
+		(pts
 			(xy 82.55 129.54) (xy 82.55 142.24)
 		)
@@
 	(wire
 		(pts
+			(xy 218.44 62.23) (xy 223.52 62.23)
+		)
+		(stroke
+			(width 0)
+			(type default)
+		)
+	)
+	(wire
+		(pts
 			(xy 257.81 114.3) (xy 264.16 114.3)
 		)
@@
 	(wire
 		(pts
-			(xy 208.28 62.23) (xy 223.52 62.23)
+			(xy 208.28 62.23) (xy 210.82 62.23)
 		)
 		(stroke
@@
 	(wire
 		(pts
+			(xy 69.85 39.37) (xy 69.85 45.72)
+		)
+		(stroke
+			(width 0)
+			(type default)
+		)
+	)
+	(wire
+		(pts
 			(xy 60.96 149.86) (xy 74.93 149.86)
 		)
@@
 	(wire
 		(pts
+			(xy 69.85 27.94) (xy 76.2 27.94)
+		)
+		(stroke
+			(width 0)
+			(type default)
+		)
+	)
+	(wire
+		(pts
 			(xy 30.48 130.81) (xy 30.48 143.51)
 		)
@@
 		)
 	)
+	(label "3V3ESP"
+		(at 76.2 27.94 0)
+		(effects
+			(font
+				(size 1.27 1.27)
+			)
+			(justify left bottom)
+		)
+	)
 	(label "3V3"
 		(at 208.28 62.23 180)
@@
 		)
 	)
+	(label "3V3ESP"
+		(at 168.91 127 0)
+		(effects
+			(font
+				(size 1.27 1.27)
+			)
+			(justify left bottom)
+		)
+	)
 	(label "22.5792"
 		(at 209.55 116.84 180)
@@
 	)
 	(label "3V3"
-		(at 72.39 45.72 0)
+		(at 77.47 45.72 0)
 		(effects
 			(font
@@
 			)
 		)
-		(property "Value" "TPS7A"
+		(property "Value" "TPS7A2033*"
 			(at 48.26 38.1 0)
 			(effects
@@
 			)
 		)
-		(property "Value" "0R68"
+		(property "Value" "0R68*"
 			(at 113.03 39.37 90)
 			(effects
@@
 	(symbol
 		(lib_id "Device:R")
+		(at 69.85 35.56 0)
+		(unit 1)
+		(exclude_from_sim no)
+		(in_bom yes)
+		(on_board yes)
+		(dnp no)
+		(fields_autoplaced yes)
+		(property "Reference" "R1"
+			(at 72.39 34.2899 0)
+			(effects
+				(font
+					(size 1.27 1.27)
+				)
+				(justify left)
+			)
+		)
+		(property "Value" "0R*"
+			(at 72.39 36.8299 0)
+			(effects
+				(font
+					(size 1.27 1.27)
+				)
+				(justify left)
+			)
+		)
+		(property "Footprint" "Resistor_SMD:R_0805_2012Metric_Pad1.20x1.40mm_HandSolder"
+			(at 68.072 35.56 90)
+			(effects
+				(font
+					(size 1.27 1.27)
+				)
+				(hide yes)
+			)
+		)
+		(property "Datasheet" "~"
+			(at 69.85 35.56 0)
+			(effects
+				(font
+					(size 1.27 1.27)
+				)
+				(hide yes)
+			)
+		)
+		(property "Description" "Resistor"
+			(at 69.85 35.56 0)
+			(effects
+				(font
+					(size 1.27 1.27)
+				)
+				(hide yes)
+			)
+		)
+		(pin "1"
+		)
+		(pin "2"
+		)
+		(instances
+			(project ""
+				(path "/4e8ba15a-9575-47ae-b6a2-ab0ac9268e83"
+					(reference "R1")
+					(unit 1)
+				)
+			)
+		)
+	)
+	(symbol
+		(lib_id "Device:R")
 		(at 87.63 135.89 0)
 		(unit 1)
@@
 	)
 	(symbol
+		(lib_id "Device:R")
+		(at 214.63 62.23 90)
+		(unit 1)
+		(exclude_from_sim no)
+		(in_bom yes)
+		(on_board yes)
+		(dnp no)
+		(property "Reference" "R11"
+			(at 210.566 61.214 90)
+			(effects
+				(font
+					(size 1.27 1.27)
+				)
+			)
+		)
+		(property "Value" "10K"
+			(at 214.63 62.23 90)
+			(effects
+				(font
+					(size 1.27 1.27)
+				)
+			)
+		)
+		(property "Footprint" "Resistor_SMD:R_0603_1608Metric_Pad0.98x0.95mm_HandSolder"
+			(at 214.63 64.008 90)
+			(effects
+				(font
+					(size 1.27 1.27)
+				)
+				(hide yes)
+			)
+		)
+		(property "Datasheet" "~"
+			(at 214.63 62.23 0)
+			(effects
+				(font
+					(size 1.27 1.27)
+				)
+				(hide yes)
+			)
+		)
+		(property "Description" "Resistor"
+			(at 214.63 62.23 0)
+			(effects
+				(font
+					(size 1.27 1.27)
+				)
+				(hide yes)
+			)
+		)
+		(pin "2"
+		)
+		(pin "1"
+		)
+		(instances
+			(project "ESP32USBI2S"
+				(path "/4e8ba15a-9575-47ae-b6a2-ab0ac9268e83"
+					(reference "R11")
+					(unit 1)
+				)
+			)
+		)
+	)
+	(symbol
 		(lib_id "Device:C")
 		(at 257.81 124.46 0)
@@
 			)
 		)
-		(property "Value" "220uF"
+		(property "Value" "220uF*"
 			(at 124.46 47.3709 0)
 			(effects
@@
 			)
 		)
-		(property "Value" "100nF"
+		(property "Value" "100nF*"
 			(at 107.95 48.2599 0)
 			(effects
@@
 			)
 		)
-		(property "Value" "100nF"
+		(property "Value" "100nF*"
 			(at 133.35 48.2599 0)
 			(effects
@@
 			)
 		)
-		(property "Value" "1uF"
+		(property "Value" "1uF*"
 			(at 146.05 48.2599 0)
 			(effects
@@
 			)
 		)
-		(property "Value" "1uF"
+		(property "Value" "1uF*"
 			(at 66.04 50.7999 0)
 			(effects
@@
 			)
 		)
-		(property "Value" "1uF"
+		(property "Value" "1uF*"
 			(at 50.8 25.3999 0)
 			(effects
@@
 			)
 		)
-		(property "Value" "220uF"
+		(property "Value" "220uF*"
 			(at 96.52 47.3709 0)
 			(effects
