File: ESP32USBI2S/ESP32USBI2S.kicad_pcb (KiCad board)
At the start: 2 copper layers, 54.9 x 67.3 mm, 34 parts, among them IC1 TPS7A, IC2 74LVC, IC3 5PB1102, J1 I2S OUT, J2 5V POWER, U1 ESP32-S3, Y2 22.5792MHz, Y3 24.5760Mhz

Commit message: final design
Parts:
- added R11: 10K, Resistor_SMD:R_0603_1608Metric_Pad0.98x0.95mm_HandSolder, F.Cu at (162.3, 88.4)
- moved R8 0.13 mm to (153.2, 90.5)
Connections:
- IC3 pad 2: /3V3 -> Net-(IC3-1G)
Routing:
- net Net-(IC3-1G): track 0.00 -> 6.51 mm
- net /3V3: track 86.0 -> 80.3 mm, vias 5 -> 4
- net GND: track 1.86 -> 3.77 mm, vias 0 -> 77
- net /LRCK: track 7.55 -> 6.83 mm
- net /DATA: track 7.55 -> 6.83 mm

Commit message: design for bare module
Parts:
- added R1: 0R*, Resistor_SMD:R_0805_2012Metric_Pad1.20x1.40mm_HandSolder, F.Cu at (137.8, 109.5)
- C2, C3, C6: value 1uF -> 1uF*
- C5, C7: value 100nF -> 100nF*
- C8, C9: value 220uF -> 220uF*
- IC1: value TPS7A -> TPS7A2033*
- R5: value 0R68 -> 0R68*
Connections:
- U1 pad 24: unconnected-(U1-3V3-Pad24) -> /3V3ESP
Routing:
- net /3V3: track 80.3 -> 115.1 mm, vias 4 -> 5
- net /3V3ESP: track 0.00 -> 5.97 mm
Other:
- board text removed: "DO NOT USE USB AND EXTERNAL POWER AT THE SAME TIME"
