File: ESP32USBITS-BARE/ESP32USBITS-BARE.kicad_sch (KiCad schematic)
At the start: 45 parts, among them IC2 74LVC, IC3 5PB1102, IC4 USBLC6, IC5 ESP32-S3-WROOM-1U-N16R8, IC6 RESET, IC7 BOOT, J1 I2S OUT, J2 Conn_01x10_Socket, J3 POWER IN, J4 USB-B CONNECTOR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

Commit message: more work
Parts:
- added J5: USB IN, Connector_Molex:Molex_KK-254_AE-6410-06A_1x06_P2.54mm_Vertical, symbol Connector:Conn_01x06_Socket
- added R17, R18: 5K1, Resistor_SMD:R_0805_2012Metric_Pad1.20x1.40mm_HandSolder, symbol Device:R
Connections:
- net GND: now also J5.1 (Pin_1), R17.2, R18.2
- net VBUS: now also J5.6 (Pin_6)
- net at IC4.6 (I/O1_2), J4.2 (D-): now also J5.2 (Pin_2)
- net at IC4.4 (I/O2_2), J4.3 (D+): now also J5.3 (Pin_3)
- new net: J5.4 (Pin_4), R18.1
- new net: J5.5 (Pin_5), R17.1
Other:
- moved on the sheet: C6, J4, R14

Commit message: more work
Parts:
- added D1, D2, D3, D4, D5: LED, LED_SMD:LED_0805_2012Metric_Pad1.15x1.40mm_HandSolder, symbol Device:LED
- added J6: COMM, Connector_PinHeader_2.54mm:PinHeader_1x04_P2.54mm_Vertical, symbol Connector:Conn_01x04_Socket
- added R19, R20: 10K, Resistor_SMD:R_0603_1608Metric_Pad0.98x0.95mm_HandSolder, symbol Device:R
- added R21, R22, R23, R24, R25: 2K2, Resistor_SMD:R_0603_1608Metric_Pad0.98x0.95mm_HandSolder, symbol Device:R
- J1, J5: footprint Connector_Molex:Molex_KK-254_AE-6410-06A_1x06_P2.54mm_Vertical -> Connector_JST:JST_XH_B6B-XH-A_1x06_P2.50mm_Vertical
Connections:
- net 3V3: now also R19.1, R20.1
- net F0: now also R21.1
- net F1: now also R22.1
- net F2: now also R23.1
- net F3: now also R24.1
- net GND: now also D1.1 (K), D2.1 (K), D3.1 (K), D4.1 (K), D5.1 (K), J6.1 (Pin_1)
- net MUTE: now also R25.1
- net SDA: now reaches IC5.12 (IO8)
- net SDA: now also J6.2 (Pin_2), R20.2
- net SCL: now reaches IC5.17 (IO9)
- net SCL: now also J6.3 (Pin_3), R19.2
- net UART: now reaches IC5.18 (IO10)
- net UART: now also J6.4 (Pin_4)
- new net: D5.2 (A), R25.2
- new net: D2.2 (A), R22.2
- new net: D4.2 (A), R24.2
- new net: D3.2 (A), R23.2
- new net: D1.2 (A), R21.2
