File: ESP32USBITS-BARE/ESP32USBITS-BARE.kicad_sch (KiCad schematic)
At the start: 61 parts, among them IC2 74LVC, IC3 5PB1102, IC4 USBLC6, IC5 ESP32-S3-WROOM-1U-N16R8, IC6 RESET, IC7 BOOT, J1 I2S OUT, J2 Conn_01x10_Socket, J3 POWER IN, J4 USB-B CONNECTOR, J5 USB IN, J6 COMM, U1 LD1117, Y2 22.5792MHz, Y3 24.5760Mhz

Commit message: more
Connections:
- net F2: now also IC5.11 (IO18); no longer IC5.30 (IO37)
- net F3: now also IC5.10 (IO17); no longer IC5.29 (IO36)
- net MUTE: now also IC5.9 (IO16); no longer IC5.28 (IO35)
Other:
- moved on the sheet: J6, R19, R20
Changed lines of the file:
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@@
 	)
 	(junction
-		(at 124.46 167.64)
+		(at 320.04 166.37)
 		(diameter 0)
 		(color 0 0 0 0)
@@
 	)
 	(junction
-		(at 130.81 170.18)
+		(at 326.39 168.91)
 		(diameter 0)
 		(color 0 0 0 0)
@@
 	(wire
 		(pts
-			(xy 118.11 165.1) (xy 135.89 165.1)
+			(xy 313.69 163.83) (xy 331.47 163.83)
 		)
 		(stroke
@@
 	(wire
 		(pts
-			(xy 124.46 161.29) (xy 124.46 167.64)
+			(xy 320.04 160.02) (xy 320.04 166.37)
 		)
 		(stroke
@@
 	(wire
 		(pts
-			(xy 124.46 143.51) (xy 124.46 153.67)
+			(xy 320.04 142.24) (xy 320.04 152.4)
 		)
 		(stroke
@@
 	(wire
 		(pts
+			(xy 110.49 101.6) (xy 135.89 101.6)
+		)
+		(stroke
+			(width 0)
+			(type default)
+		)
+	)
+	(wire
+		(pts
 			(xy 254 24.13) (xy 256.54 24.13)
 		)
@@
 	(wire
 		(pts
-			(xy 118.11 172.72) (xy 123.19 172.72)
+			(xy 313.69 171.45) (xy 318.77 171.45)
 		)
 		(stroke
@@
 	(wire
 		(pts
-			(xy 130.81 161.29) (xy 130.81 170.18)
+			(xy 326.39 160.02) (xy 326.39 168.91)
+		)
+		(stroke
+			(width 0)
+			(type default)
+		)
+	)
+	(wire
+		(pts
+			(xy 110.49 96.52) (xy 135.89 96.52)
 		)
 		(stroke
@@
 	(wire
 		(pts
-			(xy 36.83 -52.07) (xy 44.45 -52.07)
+			(xy 36.83 -52.07) (xy 54.61 -52.07)
 		)
 		(stroke
@@
 	(wire
 		(pts
-			(xy 168.91 81.28) (xy 195.58 81.28)
-		)
-		(stroke
-			(width 0)
-			(type default)
-		)
-	)
-	(wire
-		(pts
 			(xy 196.85 -74.93) (xy 196.85 -55.88)
 		)
@@
 	(wire
 		(pts
-			(xy 123.19 172.72) (xy 123.19 181.61)
-		)
-		(stroke
-			(width 0)
-			(type default)
-		)
-	)
-	(wire
-		(pts
-			(xy 168.91 86.36) (xy 195.58 86.36)
+			(xy 318.77 171.45) (xy 318.77 180.34)
 		)
 		(stroke
@@
 	(wire
 		(pts
-			(xy 130.81 170.18) (xy 135.89 170.18)
+			(xy 326.39 168.91) (xy 331.47 168.91)
 		)
 		(stroke
@@
 	(wire
 		(pts
-			(xy 124.46 167.64) (xy 135.89 167.64)
+			(xy 320.04 166.37) (xy 331.47 166.37)
 		)
 		(stroke
@@
 	(wire
 		(pts
-			(xy 168.91 83.82) (xy 195.58 83.82)
-		)
-		(stroke
-			(width 0)
-			(type default)
-		)
-	)
-	(wire
-		(pts
 			(xy 127 -49.53) (xy 139.7 -49.53)
 		)
@@
 	(wire
 		(pts
+			(xy 110.49 99.06) (xy 135.89 99.06)
+		)
+		(stroke
+			(width 0)
+			(type default)
+		)
+	)
+	(wire
+		(pts
 			(xy 223.52 119.38) (xy 231.14 119.38)
 		)
@@
 	(wire
 		(pts
-			(xy 130.81 143.51) (xy 130.81 153.67)
+			(xy 326.39 142.24) (xy 326.39 152.4)
 		)
 		(stroke
@@
 	(wire
 		(pts
-			(xy 118.11 167.64) (xy 124.46 167.64)
+			(xy 313.69 166.37) (xy 320.04 166.37)
 		)
 		(stroke
@@
 	(wire
 		(pts
-			(xy 118.11 170.18) (xy 130.81 170.18)
+			(xy 313.69 168.91) (xy 326.39 168.91)
 		)
 		(stroke
@@
 	)
 	(label "3V3"
-		(at 130.81 143.51 90)
+		(at 326.39 142.24 90)
 		(effects
 			(font
@@
 	)
 	(label "SDA"
-		(at 135.89 170.18 0)
+		(at 331.47 168.91 0)
 		(effects
 			(font
@@
 		)
 	)
+	(label "F3"
+		(at 110.49 99.06 180)
+		(effects
+			(font
+				(size 1.27 1.27)
+			)
+			(justify right bottom)
+		)
+	)
 	(label "SCL"
 		(at 110.49 116.84 180)
@@
 		)
 	)
-	(label "MUTE"
-		(at 195.58 81.28 0)
-		(effects
-			(font
-				(size 1.27 1.27)
-			)
-			(justify left bottom)
-		)
-	)
 	(label "BCLK"
 		(at 247.65 69.85 0)
@@
 	)
 	(label "VBUS"
-		(at 44.45 -52.07 0)
+		(at 54.61 -52.07 0)
 		(effects
 			(font
@@
 		)
 	)
+	(label "MUTE"
+		(at 110.49 96.52 180)
+		(effects
+			(font
+				(size 1.27 1.27)
+			)
+			(justify right bottom)
+		)
+	)
 	(label "GPIO0"
 		(at 132.08 46.99 270)
@@
 	)
 	(label "SCL"
-		(at 135.89 167.64 0)
+		(at 331.47 166.37 0)
 		(effects
 			(font
@@
 	)
 	(label "UART"
-		(at 135.89 165.1 0)
+		(at 331.47 163.83 0)
 		(effects
 			(font
@@
 		)
 	)
-	(label "F2"
-		(at 195.58 86.36 0)
-		(effects
-			(font
-				(size 1.27 1.27)
-			)
-			(justify left bottom)
-		)
-	)
 	(label "3V3"
 		(at 72.39 104.14 90)
@@
 		)
 	)
-	(label "MCLKDAC"
-		(at 208.28 29.21 180)
+	(label "F2"
+		(at 110.49 101.6 180)
 		(effects
 			(font
@@
 		)
 	)
-	(label "F3"
-		(at 195.58 83.82 0)
+	(label "MCLKDAC"
+		(at 208.28 29.21 180)
 		(effects
 			(font
 				(size 1.27 1.27)
 			)
-			(justify left bottom)
+			(justify right bottom)
 		)
 	)
@@
 	)
 	(label "3V3"
-		(at 124.46 143.51 90)
+		(at 320.04 142.24 90)
 		(effects
 			(font
@@
 	(symbol
 		(lib_id "Connector:Conn_01x04_Socket")
-		(at 113.03 170.18 180)
+		(at 308.61 168.91 180)
 		(unit 1)
 		(exclude_from_sim no)
@@
 		(fields_autoplaced yes)
 		(property "Reference" "J6"
-			(at 113.665 160.02 0)
+			(at 309.245 158.75 0)
 			(effects
 				(font
@@
 		)
 		(property "Value" "COMM"
-			(at 113.665 162.56 0)
+			(at 309.245 161.29 0)
 			(effects
 				(font
@@
 		)
 		(property "Footprint" "Connector_PinHeader_2.54mm:PinHeader_1x04_P2.54mm_Vertical"
-			(at 113.03 170.18 0)
+			(at 308.61 168.91 0)
 			(effects
 				(font
@@
 		)
 		(property "Datasheet" "~"
-			(at 113.03 170.18 0)
+			(at 308.61 168.91 0)
 			(effects
 				(font
@@
 		)
 		(property "Description" "Generic connector, single row, 01x04, script generated"
-			(at 113.03 170.18 0)
+			(at 308.61 168.91 0)
 			(effects
 				(font
@@
 	(symbol
 		(lib_id "Device:R")
-		(at 124.46 157.48 0)
+		(at 320.04 156.21 0)
 		(unit 1)
 		(exclude_from_sim no)
@@
 		(dnp no)
 		(property "Reference" "R19"
-			(at 121.666 153.924 0)
+			(at 317.246 152.654 0)
 			(effects
 				(font
@@
 		)
 		(property "Value" "10K"
-			(at 124.46 159.258 90)
+			(at 320.04 157.988 90)
 			(effects
 				(font
@@
 		)
 		(property "Footprint" "Resistor_SMD:R_0603_1608Metric_Pad0.98x0.95mm_HandSolder"
-			(at 122.682 157.48 90)
+			(at 318.262 156.21 90)
 			(effects
 				(font
@@
 		)
 		(property "Datasheet" "~"
-			(at 124.46 157.48 0)
+			(at 320.04 156.21 0)
 			(effects
 				(font
@@
 		)
 		(property "Description" "Resistor"
-			(at 124.46 157.48 0)
+			(at 320.04 156.21 0)
 			(effects
 				(font
@@
 	(symbol
 		(lib_id "Device:R")
-		(at 130.81 157.48 0)
+		(at 326.39 156.21 0)
 		(unit 1)
 		(exclude_from_sim no)
@@
 		(dnp no)
 		(property "Reference" "R20"
-			(at 128.016 153.924 0)
+			(at 323.596 152.654 0)
 			(effects
 				(font
@@
 		)
 		(property "Value" "10K"
-			(at 130.81 159.258 90)
+			(at 326.39 157.988 90)
 			(effects
 				(font
@@
 		)
 		(property "Footprint" "Resistor_SMD:R_0603_1608Metric_Pad0.98x0.95mm_HandSolder"
-			(at 129.032 157.48 90)
+			(at 324.612 156.21 90)
 			(effects
 				(font
@@
 		)
 		(property "Datasheet" "~"
-			(at 130.81 157.48 0)
+			(at 326.39 156.21 0)
 			(effects
 				(font
@@
 		)
 		(property "Description" "Resistor"
-			(at 130.81 157.48 0)
+			(at 326.39 156.21 0)
 			(effects
 				(font
@@
 	(symbol
 		(lib_id "power:GND")
-		(at 123.19 181.61 0)
+		(at 318.77 180.34 0)
 		(unit 1)
 		(exclude_from_sim no)
@@
 		(fields_autoplaced yes)
 		(property "Reference" "#PWR026"
-			(at 123.19 187.96 0)
+			(at 318.77 186.69 0)
 			(effects
 				(font
@@
 		)
 		(property "Value" "GND"
-			(at 123.19 186.69 0)
+			(at 318.77 185.42 0)
 			(effects
 				(font
@@
 		)
 		(property "Footprint" ""
-			(at 123.19 181.61 0)
+			(at 318.77 180.34 0)
 			(effects
 				(font
@@
 		)
 		(property "Datasheet" ""
-			(at 123.19 181.61 0)
+			(at 318.77 180.34 0)
 			(effects
 				(font
@@
 		)
 		(property "Description" "Power symbol creates a global label with name \"GND\" , ground"
-			(at 123.19 181.61 0)
+			(at 318.77 180.34 0)
 			(effects
 				(font
