File: ESP32USBITS-BARE/ESP32USBITS-BARE.kicad_pcb (KiCad board)
At the start: 4 copper layers, 54.9 x 67.3 mm, 47 parts, among them IC2 74LVC, IC3 5PB1102, IC4 USBLC6, IC5 ESP32-S3-WROOM-1U-N16R8, IC6 RESET, IC7 BOOT, J1 I2S OUT, J2 Conn_01x10_Socket, J3 POWER IN, J4 USB-B CONNECTOR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

Commit message: more work
Parts:
- added J5: USB IN, Connector_Molex:Molex_KK-254_AE-6410-06A_1x06_P2.54mm_Vertical, F.Cu at (157.5, 55.9)
- added R17: 5K1, Resistor_SMD:R_0805_2012Metric_Pad1.20x1.40mm_HandSolder, F.Cu at (148.8, 62.2)
- added R18: 5K1, Resistor_SMD:R_0805_2012Metric_Pad1.20x1.40mm_HandSolder, F.Cu at (150.9, 62.2)
- moved J4 0.08 mm to (149.9, 68.0)
Routing:
- net Net-(IC4-I/O1_2): track 10.7 -> 24.0 mm
- net /VBUS: track 20.3 -> 33.4 mm
- net Net-(IC4-I/O2_2): track 8.91 -> 19.1 mm
- net Net-(J5-Pin_5): track 0.00 -> 5.98 mm
- net Net-(J5-Pin_4): track 0.00 -> 5.77 mm
- net /MCLKESP: track 27.2 -> 30.8 mm
- net Net-(IC5-IO5): track 42.1 -> 45.1 mm
- net Net-(IC5-IO4): track 42.3 -> 45.4 mm
- net Net-(IC5-IO6): track 40.4 -> 43.5 mm
- net /3V3: track 184.2 -> 183.4 mm
- net GND: vias 82 -> 139
Other:
- board text added: "VBUS CC1 CC2 D+ D- GND"

Commit message: more work
Parts:
- added D1: LED, LED_SMD:LED_0805_2012Metric_Pad1.15x1.40mm_HandSolder, F.Cu at (150.6, 105.9)
- added D2: LED, LED_SMD:LED_0805_2012Metric_Pad1.15x1.40mm_HandSolder, F.Cu at (148.1, 105.9)
- added D3: LED, LED_SMD:LED_0805_2012Metric_Pad1.15x1.40mm_HandSolder, F.Cu at (145.5, 105.9)
- added D4: LED, LED_SMD:LED_0805_2012Metric_Pad1.15x1.40mm_HandSolder, F.Cu at (143.0, 105.9)
- added D5: LED, LED_SMD:LED_0805_2012Metric_Pad1.15x1.40mm_HandSolder, F.Cu at (140.5, 105.9)
- added J6: COMM, Connector_PinHeader_2.54mm:PinHeader_1x04_P2.54mm_Vertical, F.Cu at (135.4, 87.4)
- added R19: 10K, Resistor_SMD:R_0603_1608Metric_Pad0.98x0.95mm_HandSolder, F.Cu at (139.8, 94.8)
- added R20: 10K, Resistor_SMD:R_0603_1608Metric_Pad0.98x0.95mm_HandSolder, F.Cu at (139.6, 88.1)
- added R21: 2K2, Resistor_SMD:R_0603_1608Metric_Pad0.98x0.95mm_HandSolder, F.Cu at (150.6, 109.7)
- added R22: 2K2, Resistor_SMD:R_0603_1608Metric_Pad0.98x0.95mm_HandSolder, F.Cu at (148.1, 109.7)
- added R23: 2K2, Resistor_SMD:R_0603_1608Metric_Pad0.98x0.95mm_HandSolder, F.Cu at (145.5, 109.7)
- added R24: 2K2, Resistor_SMD:R_0603_1608Metric_Pad0.98x0.95mm_HandSolder, F.Cu at (143.0, 109.7)
- added R25: 2K2, Resistor_SMD:R_0603_1608Metric_Pad0.98x0.95mm_HandSolder, F.Cu at (140.5, 109.7)
- J1, J5: footprint Connector_Molex:Molex_KK-254_AE-6410-06A_1x06_P2.54mm_Vertical -> Connector_JST:JST_XH_B6B-XH-A_1x06_P2.50mm_Vertical
- moved G*** 45.4 mm to (158.5, 108.1)
- moved G*** 40.1 mm to (125.7, 77.1)
- moved R10 5.18 mm to (140.8, 99.2)
- moved C12 2.16 mm to (133.0, 103.5)
- moved J1 0.07 mm to (124.1, 101.5)
Connections:
- IC5 pad 12: unconnected-(IC5-IO8-Pad12) -> /SDA
- IC5 pad 17: unconnected-(IC5-IO9-Pad17) -> /SCL
- IC5 pad 18: unconnected-(IC5-IO10-Pad18) -> /UART
Routing:
- net /SCL: track 0.00 -> 20.6 mm
- net /3V3: track 183.4 -> 202.2 mm, vias 8 -> 10
- net /SDA: track 0.00 -> 17.1 mm, vias 0 -> 2
- net /UART: track 0.00 -> 10.8 mm
- net /F0: track 15.0 -> 19.5 mm
- net /F1: track 14.7 -> 19.2 mm
- net /MUTE: track 21.0 -> 25.5 mm
- net /F3: track 18.5 -> 23.0 mm
- net /F2: track 16.3 -> 20.8 mm
- net Net-(IC3-Y1): track 5.02 -> 2.72 mm
- net /MCLKESP: track 30.8 -> 28.9 mm
- net Net-(D4-A): track 0.00 -> 1.88 mm
- net Net-(D3-A): track 0.00 -> 1.88 mm
- net Net-(D2-A): track 0.00 -> 1.88 mm
- net Net-(D5-A): track 0.00 -> 1.87 mm
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Other:
- board text added: "ESP32-S3 USB to I2S - 96KHz/24bit - Self Powered © Tom Watson Audio 2026"
- board text added: "URT SCL SDA GND"
- board text removed: "ESP32-S3 USB to I2S Bridge - Self Powered © Tom Watson Audio 2026"

Commit message: ok
Routing:
- net /SCL: track 20.6 -> 22.0 mm
- net GND: vias 151 -> 155
Other:
- board text added: "5V GND"
Changed lines of the file:
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@@
 			(at 1.25 4.6 0)
 			(layer "F.SilkS")
+			(hide yes)
 			(effects
 				(font
@@
 		)
 		(property "Value" "100nF"
-			(at 4.318 0 0)
+			(at 3.937 0 0)
 			(layer "F.SilkS")
 			(effects
@@
 		)
 	)
+	(gr_text "5V  GND"
+		(at 130.302 53.086 0)
+		(layer "F.SilkS")
+		(effects
+			(font
+				(size 0.6 0.6)
+				(thickness 0.087)
+			)
+		)
+	)
 	(gr_text "F1"
 		(at 148.1328 112.903 0)
@@
 	)
 	(via
-		(at 118.11 114.3)
+		(at 118.11 115.062)
 		(size 0.6)
 		(drill 0.3)
@@
 	)
 	(via
-		(at 118.11 109.22)
+		(at 118.11 109.982)
 		(size 0.6)
 		(drill 0.3)
@@
 	)
 	(via
-		(at 118.11 106.68)
+		(at 118.11 107.188)
 		(size 0.6)
 		(drill 0.3)
@@
 	)
 	(via
-		(at 118.11 111.76)
+		(at 118.11 112.522)
 		(size 0.6)
 		(drill 0.3)
@@
 	)
 	(via
+		(at 160.274 103.124)
+		(size 0.6)
+		(drill 0.3)
+		(layers "F.Cu" "B.Cu")
+		(free yes)
+		(net 28)
+	)
+	(via
 		(at 118.11 53.34)
 		(size 0.6)
@@
 	)
 	(via
+		(at 160.274 99.568)
+		(size 0.6)
+		(drill 0.3)
+		(layers "F.Cu" "B.Cu")
+		(free yes)
+		(net 28)
+	)
+	(via
 		(at 165.1 72.39)
 		(size 0.6)
@@
 	)
 	(via
+		(at 162.306 99.568)
+		(size 0.6)
+		(drill 0.3)
+		(layers "F.Cu" "B.Cu")
+		(free yes)
+		(net 28)
+	)
+	(via
 		(at 151.13 116.84)
 		(size 0.6)
@@
 	)
 	(via
-		(at 118.11 104.14)
+		(at 162.56 103.124)
+		(size 0.6)
+		(drill 0.3)
+		(layers "F.Cu" "B.Cu")
+		(free yes)
+		(net 28)
+	)
+	(via
+		(at 118.11 104.394)
 		(size 0.6)
 		(drill 0.3)
@@
 	)
 	(via
-		(at 118.11 101.6)
+		(at 118.11 102.108)
 		(size 0.6)
 		(drill 0.3)
@@
 	)
 	(segment
-		(start 137.613 96.147)
-		(end 134.90524 96.147)
+		(start 138.731 93.933)
+		(end 136.398 96.266)
+		(width 0.2)
+		(layer "F.Cu")
+		(net 54)
+	)
+	(segment
+		(start 133.858 95.758)
+		(end 133.858 92.964)
 		(width 0.2)
 		(layer "F.Cu")
@@
 	)
 	(segment
-		(start 134.231 93.607)
+		(start 134.366 92.456)
 		(end 135.382 92.456)
 		(width 0.2)
@@
 	(segment
 		(start 139.827 93.933)
-		(end 137.613 96.147)
+		(end 138.731 93.933)
 		(width 0.2)
 		(layer "F.Cu")
@@
 	)
 	(segment
-		(start 134.90524 96.147)
-		(end 134.231 95.47276)
+		(start 134.366 96.266)
+		(end 133.858 95.758)
+		(width 0.2)
+		(layer "F.Cu")
+		(net 54)
+	)
+	(segment
+		(start 136.398 96.266)
+		(end 134.366 96.266)
 		(width 0.2)
 		(layer "F.Cu")
@@
 	)
 	(segment
-		(start 134.231 95.47276)
-		(end 134.231 93.607)
+		(start 133.858 92.964)
+		(end 134.366 92.456)
 		(width 0.2)
 		(layer "F.Cu")
