File: ESP32USBITS-BARE/ESP32USBITS-BARE.kicad_pcb (KiCad board)
At the start: 4 copper layers, 54.9 x 67.3 mm, 63 parts, among them IC2 74LVC, IC3 5PB1102, IC4 USBLC6, IC5 ESP32-S3-WROOM-1U-N16R8, IC6 RESET, IC7 BOOT, J1 I2S OUT, J2 Conn_01x10_Socket, J3 POWER IN, J4 USB-B CONNECTOR, J5 USB IN, J6 COMM, U1 LD1117, Y2 22.5792MHz, Y3 24.5760Mhz

Commit message: more
Connections:
- IC5 pad 10: unconnected-(IC5-IO17-Pad10) -> /F3
- IC5 pad 11: unconnected-(IC5-IO18-Pad11) -> /F2
- IC5 pad 28: /MUTE -> unconnected-(IC5-IO35-Pad28)
- IC5 pad 29: /F3 -> unconnected-(IC5-IO36-Pad29)
- IC5 pad 30: /F2 -> unconnected-(IC5-IO37-Pad30)
- IC5 pad 9: unconnected-(IC5-IO16-Pad9) -> /MUTE
Routing:
- net /MUTE: track 25.5 -> 44.9 mm
- net /F3: track 23.0 -> 41.4 mm
- net /F2: track 20.8 -> 38.3 mm
- net /3V3: track 202.2 -> 202.8 mm
Changed lines of the file:
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@@
 	(net 22 "unconnected-(IC5-IO3-Pad15)")
 	(net 23 "unconnected-(IC5-IO48-Pad25)")
-	(net 24 "unconnected-(IC5-IO16-Pad9)")
+	(net 24 "unconnected-(IC5-IO37-Pad30)")
 	(net 25 "/F2")
 	(net 26 "unconnected-(IC5-IO45-Pad26)")
@@
 	(net 47 "Net-(IC3-Y0)")
 	(net 48 "Net-(IC3-1G)")
-	(net 49 "unconnected-(IC5-IO18-Pad11)")
-	(net 50 "unconnected-(IC5-IO17-Pad10)")
+	(net 49 "unconnected-(IC5-IO35-Pad28)")
+	(net 50 "unconnected-(IC5-IO36-Pad29)")
 	(net 51 "unconnected-(IC5-IO47-Pad24)")
 	(net 52 "unconnected-(IC5-IO14-Pad22)")
@@
 			(size 0.9 1.5)
 			(layers "F.Cu" "F.Mask" "F.Paste")
-			(net 24 "unconnected-(IC5-IO16-Pad9)")
+			(net 32 "/MUTE")
 			(pinfunction "IO16")
 			(pintype "passive")
@@
 			(size 0.9 1.5)
 			(layers "F.Cu" "F.Mask" "F.Paste")
-			(net 50 "unconnected-(IC5-IO17-Pad10)")
+			(net 17 "/F3")
 			(pinfunction "IO17")
 			(pintype "passive")
@@
 			(size 0.9 1.5)
 			(layers "F.Cu" "F.Mask" "F.Paste")
-			(net 49 "unconnected-(IC5-IO18-Pad11)")
+			(net 25 "/F2")
 			(pinfunction "IO18")
 			(pintype "passive")
@@
 			(size 0.9 1.5)
 			(layers "F.Cu" "F.Mask" "F.Paste")
-			(net 32 "/MUTE")
+			(net 49 "unconnected-(IC5-IO35-Pad28)")
 			(pinfunction "IO35")
 			(pintype "passive")
@@
 			(size 0.9 1.5)
 			(layers "F.Cu" "F.Mask" "F.Paste")
-			(net 17 "/F3")
+			(net 50 "unconnected-(IC5-IO36-Pad29)")
 			(pinfunction "IO36")
 			(pintype "passive")
@@
 			(size 0.9 1.5)
 			(layers "F.Cu" "F.Mask" "F.Paste")
-			(net 25 "/F2")
+			(net 24 "unconnected-(IC5-IO37-Pad30)")
 			(pinfunction "IO37")
 			(pintype "passive")
@@
 	)
 	(segment
-		(start 147.701 103.124)
-		(end 147.701 101.32)
+		(start 148.321 91.948)
+		(end 149.002654 91.948)
+		(width 0.3)
+		(layer "F.Cu")
+		(net 17)
+	)
+	(segment
+		(start 149.86 91.090654)
+		(end 149.86 84.201)
+		(width 0.3)
+		(layer "F.Cu")
+		(net 17)
+	)
+	(segment
+		(start 149.86 84.201)
+		(end 150.241 83.82)
 		(width 0.3)
 		(layer "F.Cu")
@@
 		(net 17)
 	)
+	(segment
+		(start 149.002654 91.948)
+		(end 149.86 91.090654)
+		(width 0.3)
+		(layer "F.Cu")
+		(net 17)
+	)
 	(via
-		(at 147.701 103.124)
+		(at 148.321 91.948)
 		(size 0.6)
 		(drill 0.3)
@@
 	)
 	(segment
+		(start 148.47 103.893)
+		(end 148.47 92.097)
+		(width 0.3)
+		(layer "B.Cu")
+		(net 17)
+	)
+	(segment
 		(start 147.377009 113.41551)
 		(end 148.3616 113.41551)
@@
 	)
 	(segment
-		(start 148.47 103.893)
-		(end 147.701 103.124)
+		(start 148.47 92.097)
+		(end 148.321 91.948)
 		(width 0.3)
 		(layer "B.Cu")
@@
 	)
 	(segment
-		(start 145.542 110.6405)
-		(end 145.542 115.11751)
+		(start 148.971 91.059)
+		(end 148.971 83.82)
 		(width 0.3)
 		(layer "F.Cu")
@@
 	)
 	(segment
-		(start 148.971 103.124)
-		(end 148.971 101.32)
+		(start 145.542 110.6405)
+		(end 145.542 115.11751)
 		(width 0.3)
 		(layer "F.Cu")
@@
 	)
 	(via
-		(at 148.971 103.124)
+		(at 148.971 91.059)
 		(size 0.6)
 		(drill 0.3)
@@
 	)
 	(segment
+		(start 148.971 103.124)
+		(end 148.971 91.059)
+		(width 0.3)
+		(layer "B.Cu")
+		(net 25)
+	)
+	(segment
 		(start 145.542 115.11751)
 		(end 146.383529 115.11751)
@@
 	)
 	(via
+		(at 151.13 90.297)
+		(size 0.6)
+		(drill 0.3)
+		(layers "F.Cu" "B.Cu")
+		(free yes)
+		(net 28)
+	)
+	(via
 		(at 137.16 53.34)
 		(size 0.6)
@@
 	)
 	(via
-		(at 151.003 90.17)
-		(size 0.6)
-		(drill 0.3)
-		(layers "F.Cu" "B.Cu")
-		(free yes)
-		(net 28)
-	)
-	(via
 		(at 156.591 90.678)
 		(size 0.6)
@@
 	)
 	(segment
-		(start 146.431 103.124)
-		(end 146.431 101.32)
+		(start 147.574 92.456)
+		(end 147.717 92.599)
+		(width 0.3)
+		(layer "F.Cu")
+		(net 32)
+	)
+	(segment
+		(start 147.717 92.599)
+		(end 149.060174 92.599)
 		(width 0.3)
 		(layer "F.Cu")
@@
 		(net 32)
 	)
+	(segment
+		(start 150.361 85.602)
+		(end 151.511 84.452)
+		(width 0.3)
+		(layer "F.Cu")
+		(net 32)
+	)
+	(segment
+		(start 150.361 91.298174)
+		(end 150.361 85.602)
+		(width 0.3)
+		(layer "F.Cu")
+		(net 32)
+	)
+	(segment
+		(start 151.511 84.452)
+		(end 151.511 83.82)
+		(width 0.3)
+		(layer "F.Cu")
+		(net 32)
+	)
+	(segment
+		(start 149.060174 92.599)
+		(end 150.361 91.298174)
+		(width 0.3)
+		(layer "F.Cu")
+		(net 32)
+	)
 	(via
-		(at 146.431 103.124)
+		(at 147.574 92.456)
 		(size 0.6)
 		(drill 0.3)
@@
 	(segment
 		(start 147.969 104.10052)
-		(end 147.64348 103.775)
+		(end 147.969 92.851)
 		(width 0.3)
 		(layer "B.Cu")
@@
 	)
 	(segment
-		(start 147.64348 103.775)
-		(end 147.082 103.775)
+		(start 141.303529 115.11751)
+		(end 142.504529 113.91651)
 		(width 0.3)
 		(layer "B.Cu")
@@
 	)
 	(segment
-		(start 141.303529 115.11751)
-		(end 142.504529 113.91651)
+		(start 147.969 92.851)
+		(end 147.574 92.456)
 		(width 0.3)
 		(layer "B.Cu")
@@
 	)
 	(segment
-		(start 147.082 103.775)
-		(end 146.431 103.124)
-		(width 0.3)
-		(layer "B.Cu")
-		(net 32)
-	)
-	(segment
 		(start 144.837009 113.41551)
 		(end 146.668489 113.41551)
@@
 	)
 	(segment
-		(start 125.222 86.487)
-		(end 126.746 84.963)
+		(start 125.222 85.471)
+		(end 125.73 84.963)
 		(width 0.3)
 		(layer "In2.Cu")
@@
 	)
 	(segment
-		(start 125.222 94.361)
-		(end 125.222 86.487)
+		(start 125.73 84.963)
+		(end 126.746 84.963)
 		(width 0.3)
 		(layer "In2.Cu")
@@
 		(layer "In2.Cu")
 		(net 36)
+	)
+	(segment
+		(start 125.222 94.361)
+		(end 125.222 85.471)
+		(width 0.3)
+		(layer "In2.Cu")
+		(net 36)
